File: Kicad/Riser_M19_EXT.kicad_pcb (KiCad board)
At the start: 2 copper layers, 102 x 105.7 mm, 18 parts

Commit message: Rev 1.2
Routing:
- added copper zone on B.Cu, net GND
- added copper zone on F.Cu, net GND
- removed copper zone on B.Cu, net VCC
- removed copper zone on F.Cu, net VCC
Other:
- board text added: "M19 External Riser PSU V 1.2"
- board text removed: "M19 External Riser PSU V 1.1"
Changed lines of the file:
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@@
 		(layer "B.Fab")
 	)
-	(gr_text "M19 External Riser PSU V 1.1"
+	(gr_text "M19 External Riser PSU V 1.2"
 		(at 123.86 38.9 0)
 		(layer "F.SilkS")
@@
 		(start 193.04 135.382)
 		(end 193.04 107.95)
-		(width 0.6)
+		(width 1)
 		(layer "B.Cu")
 		(net 9)
@@
 		(start 116.84 96.52)
 		(end 116.84 135.382)
-		(width 0.6)
+		(width 1)
 		(layer "B.Cu")
 		(net 9)
@@
 		(start 170.18 135.382)
 		(end 170.18 95.25)
-		(width 0.4)
+		(width 1)
 		(layer "B.Cu")
 		(net 9)
@@
 	)
 	(zone
-		(net 12)
-		(net_name "VCC")
-		(layers "F.Cu" "B.Cu")
-		(hatch edge 0.5)
-		(connect_pads
-			(clearance 0.5)
-		)
-		(min_thickness 0.25)
-		(filled_areas_thickness no)
-		(fill yes
-			(thermal_gap 0.5)
-			(thermal_bridge_width 0.5)
-		)
-		(polygon
-			(pts
-				(xy 115.57 129.54) (xy 194.31 129.54) (xy 194.31 111.76) (xy 196.85 111.76) (xy 198.12 110.49) (xy 198.12 35.56)
-				(xy 97.79 35.56) (xy 97.79 110.49) (xy 99.06 111.76) (xy 115.57 111.76)
-			)
-		)
-	)
-	(zone
 		(net 0)
 		(net_name "")
@@
 			)
 		)
+	)
+	(zone
+		(net 9)
+		(net_name "GND")
+		(layers "F.Cu" "B.Cu")
+		(hatch edge 0.5)
+		(connect_pads
+			(clearance 0.5)
+		)
+		(min_thickness 0.25)
+		(filled_areas_thickness no)
+		(fill yes
+			(thermal_gap 0.5)
+			(thermal_bridge_width 0.5)
+		)
+		(polygon
+			(pts
+				(xy 97.79 34.925) (xy 198.12 34.925) (xy 198.12 111.76) (xy 194.945 111.76) (xy 194.945 130.81)
+				(xy 114.935 130.81) (xy 114.935 111.76) (xy 97.79 111.76)
+			)
+		)
